Commit message: fix: Fix continuous joints limits

File: config/urdfs/kortex.urdf (robot description, URDF)
Before this commit: robot gen3_robotiq_2f_85, 24 links, 23 joints
Joints:
- joint joint_1: limit lower=-3.14 upper=3.14 effort=39 velocity=1.3963 -> effort=39 velocity=1.3963
- joint joint_3: limit lower=-3.14 upper=3.14 effort=39 velocity=1.3963 -> effort=39 velocity=1.3963
- joint joint_5: limit lower=-3.14 upper=3.14 effort=9 velocity=1.2218 -> effort=9 velocity=1.2218
- joint joint_7: limit lower=-3.14 upper=3.14 effort=9 velocity=1.2218 -> effort=9 velocity=1.2218
