Commit message: fix: IONA (chest + right arm)

File: config/urdfs/iona_right_arm.urdf (robot description, URDF)
Before this commit: robot iona_right_arm, 24 links, 23 joints
Links:
- removed link right_arm_mount
- added link chest_link_fixed
Joints:
- removed joint chest_to_right_arm_mount
- removed joint right_arm_mount_to_arm
- added joint chest_joint_fixed: type fixed, parent chest_link, child chest_link_fixed, origin xyz=0 0 0 rpy=0 0 0
- added joint chest_to_right_base: type fixed, parent chest_link_fixed, child right/base_link, origin xyz=0.0 -0.142 -0.038 rpy=0.0 0.7829999999999999 -1.5659999999999998
- joint chest_joint: origin xyz=0 0 0.5775 rpy=0 0 0 -> xyz=0 0 0.5775 rpy=0 0 3.14
- joint right/joint_1: limit lower=-3.14 upper=3.14 effort=39 velocity=1.3963 -> lower=-6.28 upper=6.28 effort=39 velocity=1.3963
- joint right/joint_3: limit lower=-3.14 upper=3.14 effort=39 velocity=1.3963 -> lower=-6.28 upper=6.28 effort=39 velocity=1.3963
- joint right/joint_5: limit lower=-3.14 upper=3.14 effort=9 velocity=1.2218 -> lower=-6.28 upper=6.28 effort=9 velocity=1.2218
- joint right/joint_7: limit lower=-3.14 upper=3.14 effort=9 velocity=1.2218 -> lower=-6.28 upper=6.28 effort=9 velocity=1.2218
